Commit message: chore: Update URDF for c_moveit_config
This commit updates the URDF files for the c_moveit_config package. The changes include:
- Adding a settings.json file to the robotiq_hande_description package with the "ros.distro" set to "jazzy".
- Deleting the settings.json file from the robotiq_description package.
- Adding a c_bot_hw.yaml file to the noetic_ur/noetic_fake/config directory with various settings for the ros_control hardware interface.
- Adding a load_robotiq_hande.launch file to the robotiq_hande_description/launch directory, which includes the robotiq_hande.xacro file and sets the transmission_hw_interface argument.
- Deleting the load_robotiq_hande.launch file from the robotiq_description/launch directory.
- Adding a c_bot_calibration.launch file to the noetic_ur/noetic_bringup/launch directory, which includes the calibration_correction.launch file from the ur_calibration package.
- Adding a c_bot_moveit_controllers.yaml file to the noetic_ur/noetic_gazebo/config directory, which defines the controllers for the c_bot in Gazebo.
- Adding a c_bot_moveit_controllers.yaml file to the noetic_ur/noetic_bringup/config directory, which defines the controllers for the c_bot in MoveIt.
- Adding a c_bot_moveit_controllers.yaml file to the noetic_ur/noetic_fake/config directory, which defines the controllers for the c_bot in the fake hardware interface.
- Adding a view_robotiq_hande.launch file to the robotiq_hande_description/launch directory, which includes the load_robotiq_hande.launch file and launches the joint_state_publisher_gui, robot_state_publisher, and rviz nodes.

These changes were made to update the URDF and launch files for the c_moveit_config package, improving the functionality and compatibility of the robotiq_hande_description package.

File: catkin_ws/src/noetic_ur/noetic_c_bot_moveit_config/config/gazebo_c_bot_scene.urdf (robot description, URDF)
Before this commit: robot c_bot_scene, 31 links, 30 joints
Links:
- link gripper_body: geometry collision mesh filename=package://robotiq_hande_description/meshes/hande/hand-e-col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 scale=1.0 1.0 1.0; visual mesh filename=package://robotiq_hande_description/meshes/hande/hand-e.dae scale=1.0 1.0 1.0
- link hande_left_finger: geometry collision mesh filename=package://robotiq_hande_description/meshes/hande/finger_1-c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 scale=1.0 1.0 1.0; visual mesh filename=package://robotiq_hande_description/meshes/hande/finger_1.d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 scale=1.0 1.0 1.0
- link hande_right_finger: geometry collision mesh filename=package://robotiq_hande_description/meshes/hande/finger_2-c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 scale=1.0 1.0 1.0; visual mesh filename=package://robotiq_hande_description/meshes/hande/finger_2.d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 scale=1.0 1.0 1.0

File: catkin_ws/src/noetic_ur/noetic_description/urdf/macros/c_bot_macro.xacro (robot description, xacro)
@@ -4,5 +4,5 @@
     <xacro:include filename="$(find noetic_description)/urdf/macros/d415_mount_macro.xacro" />
     <xacro:include
-        filename="$(find robotiq_description)/urdf/robotiq_hande_macro.xacro" />
+        filename="$(find robotiq_hande_description)/urdf/robotiq_hande_macro.xacro" />
     <xacro:macro name="c_bot"
         params="

File: catkin_ws/src/robotiq/robotiq_hande_description/urdf/robotiq_hande_macro.xacro (robot description, xacro)
@@ -2,7 +2,7 @@
 <robot xmlns:xacro="http://ros.org/wiki/xacro">
   <xacro:include
-    filename="$(find robotiq_description)/urdf/inc/robotiq_hande.transmissions.xacro" />
+    filename="$(find robotiq_hande_description)/urdf/inc/robotiq_hande.transmissions.xacro" />
   <xacro:include
-    filename="$(find robotiq_description)/urdf/inc/robotiq_hande_gazebo.xacro" />
+    filename="$(find robotiq_hande_description)/urdf/inc/robotiq_hande_gazebo.xacro" />
   <xacro:macro name="robotiq_hande"
     params="
@@ -23,5 +23,5 @@
         <origin rpy="0 0 0" xyz="0 0 0"/>
         <geometry>
-          <mesh filename="package://robotiq_description/meshes/hande/finger_1.dae" scale="1.0 1.0 1.0"/>
+          <mesh filename="package://robotiq_hande_description/meshes/hande/finger_1.dae" scale="1.0 1.0 1.0"/>
         </geometry>
         <material name="DarkGray">
@@ -32,5 +32,5 @@
         <origin rpy="0 0 0" xyz="0 0 0"/>
         <geometry>
-          <mesh filename="package://robotiq_description/meshes/hande/finger_1-collision.dae" scale="1.0 1.0 1.0"/>
+          <mesh filename="package://robotiq_hande_description/meshes/hande/finger_1-collision.dae" scale="1.0 1.0 1.0"/>
         </geometry>
       </collision>
@@ -45,5 +45,5 @@
         <origin rpy="0 0 0" xyz="0 0 0"/>
         <geometry>
-          <mesh filename="package://robotiq_description/meshes/hande/finger_2.dae" scale="1.0 1.0 1.0"/>
+          <mesh filename="package://robotiq_hande_description/meshes/hande/finger_2.dae" scale="1.0 1.0 1.0"/>
         </geometry>
         <material name="DarkGray">
@@ -54,5 +54,5 @@
         <origin rpy="0 0 0" xyz="0 0 0"/>
         <geometry>
-          <mesh filename="package://robotiq_description/meshes/hande/finger_2-collision.dae" scale="1.0 1.0 1.0"/>
+          <mesh filename="package://robotiq_hande_description/meshes/hande/finger_2-collision.dae" scale="1.0 1.0 1.0"/>
         </geometry>
       </collision>
@@ -155,5 +155,5 @@
         <origin rpy="0 0 0" xyz="0 0 0"/>
         <geometry>
-          <mesh filename="package://robotiq_description/meshes/hande/hand-e.dae" scale="1.0 1.0 1.0"/>
+          <mesh filename="package://robotiq_hande_description/meshes/hande/hand-e.dae" scale="1.0 1.0 1.0"/>
         </geometry>
         <material name="Dark">
@@ -164,5 +164,5 @@
         <origin rpy="0 0 0" xyz="0 0 0"/>
         <geometry>
-          <mesh filename="package://robotiq_description/meshes/hande/hand-e-collision.dae" scale="1.0 1.0 1.0"/>
+          <mesh filename="package://robotiq_hande_description/meshes/hande/hand-e-collision.dae" scale="1.0 1.0 1.0"/>
         </geometry>
       </collision>
