Commit message: Refactor gripper parameters in launch and source files

File: sim/catkin_ws/src/robotiq/robotiq_hande_description/urdf/robotiq_hande_macro.xacro (robot description, xacro)
@@ -12,6 +12,6 @@
       hw_interface="${transmission_hw_interface}" />
     <xacro:robotiq_hande_gazebo prefix="${prefix}" />
-    <xacro:property name="max_effort" value="130.0" />
-    <xacro:property name="max_velocity" value="2.0" />
+    <xacro:property name="max_effort" value="185.0" />
+    <xacro:property name="max_velocity" value="0.15" />
     <link name="${prefix}hande_left_finger">
       <inertial>
@@ -63,5 +63,5 @@
       <child link="${prefix}hande_left_finger"/>
       <axis xyz="-1 0 0"/>
-      <limit effort="130" lower="0" upper="0.025" velocity="0.15"/>
+      <limit effort="185" lower="0" upper="0.025" velocity="0.15"/>
     </joint>
     <joint name="${prefix}hande_right_finger_joint" type="prismatic">
@@ -70,5 +70,5 @@
       <child link="${prefix}hande_right_finger"/>
       <axis xyz="1 0 0"/>
-      <limit effort="130" lower="0" upper="0.025" velocity="0.15"/>
+      <limit effort="185" lower="0" upper="0.025" velocity="0.15"/>
       <mimic joint="${prefix}hande_left_finger_joint" multiplier="1" offset="0"/>
     </joint>
